Commit message: working (barely) camera feed and cleaned up other launch files

File: ros2_ws/src/libra/models/camera.urdf (robot description, URDF)
Before this commit: robot sensor_suites, 2 links, 1 joints
Links:
- removed link base_link
- added link camera_frame; collision box size=${camera_length} ${camera_width} ${camera_height}; visual box size=${camera_length} ${camera_width} ${camera_height}
Joints:
- joint base_joint: child base_link -> camera_frame
